Commit message: urdf files fixed simple_velocity_controller broken

File: my_robot_description/urdf/mobile_base_gazebo.xacro (robot description, xacro)
@@ -8,4 +8,5 @@
     </gazebo>
     <gazebo reference="right_front_wheel_link">
+        <!-- Buraya bir sey ekledim -->
         <material>Gazebo/Grey</material>
         <mu1>10000000000000.0</mu1>

File: my_robot_description/urdf/my_robot.urdf.xacro (robot description, xacro)
@@ -3,9 +3,9 @@
     <!-- Properties -->
     <xacro:include filename="common_properties.xacro" />
+    <!-- ROS2 Control -->
+    <xacro:include filename="my_robot_ros2_control.xacro"/>
     <!-- Robot URDF -->
     <xacro:include filename="mobile_base.xacro" />
     <!-- Include Gazebo Parameters -->
     <xacro:include filename="mobile_base_gazebo.xacro" />
-    <!-- ROS2 Control -->
-    <xacro:include filename="my_robot_ros2_control.xacro"/>
 </robot>

File: my_robot_description/urdf/my_robot_ros2_control.xacro (robot description, xacro)
@@ -5,36 +5,36 @@
             <plugin>ign_ros2_control/IgnitionSystem</plugin>
         </hardware>
+        <joint name="base_right_front_wheel_joint">
+            <command_interface name="velocity">
+                <param name="min">-1</param>
+                <param name="max">1</param>
+            </command_interface>
+            <state_interface name="position"/>
+            <state_interface name="velocity"/>
+        </joint>
+        <joint name="base_right_back_wheel_joint">
+            <command_interface name="velocity">
+                <param name="min">-1</param>
+                <param name="max">1</param>
+            </command_interface>
+            <state_interface name="position"/>
+            <state_interface name="velocity"/>
+        </joint>
+        <joint name="base_left_front_wheel_joint">
+            <command_interface name="velocity">
+                <param name="min">-1</param>
+                <param name="max">1</param>
+            </command_interface>
+            <state_interface name="position"/>
+            <state_interface name="velocity"/>
+        </joint>
+        <joint name="base_left_back_wheel_joint">
+            <command_interface name="velocity">
+                <param name="min">-1</param>
+                <param name="max">1</param>
+            </command_interface>
+            <state_interface name="position"/>
+            <state_interface name="velocity"/>
+        </joint>
     </ros2_control>
-    <joint name="base_right_front_wheel_joint">
-        <command_interface name="velocity">
-            <param name="min">-1</param>
-            <param name="max">1</param>
-        </command_interface>
-        <state_interface name="position"/>
-        <state_interface name="velocity"/>
-    </joint>
-    <joint name="base_right_back_wheel_joint">
-        <command_interface name="velocity">
-            <param name="min">-1</param>
-            <param name="max">1</param>
-        </command_interface>
-        <state_interface name="position"/>
-        <state_interface name="velocity"/>
-    </joint>
-    <joint name="base_left_front_wheel_joint">
-        <command_interface name="velocity">
-            <param name="min">-1</param>
-            <param name="max">1</param>
-        </command_interface>
-        <state_interface name="position"/>
-        <state_interface name="velocity"/>
-    </joint>
-    <joint name="base_left_back_wheel_joint">
-        <command_interface name="velocity">
-            <param name="min">-1</param>
-            <param name="max">1</param>
-        </command_interface>
-        <state_interface name="position"/>
-        <state_interface name="velocity"/>
-    </joint>
 </robot>

Commit message: joystick added, robot can be driven on gazebo

File: my_robot_description/urdf/mobile_base_gazebo.xacro (robot description, xacro)
@@ -10,5 +10,5 @@
         <!-- Buraya bir sey ekledim -->
         <material>Gazebo/Grey</material>
-        <mu1>10000000000000.0</mu1>
+        <!-- <mu1>10000000000000.0</mu1>
         <mu2>10000000000000.0</mu2>
         <kp>1000000000.0</kp>
@@ -16,9 +16,9 @@
         <minDepth>0.001</minDepth>
         <maxVel>0.1</maxVel>
-        <fdir1>1 0 0</fdir1>
+        <fdir1>1 0 0</fdir1> -->
     </gazebo>
     <gazebo reference="right_back_wheel_link">
         <material>Gazebo/Grey</material>
-        <mu1>10000000000000.0</mu1>
+        <!-- <mu1>10000000000000.0</mu1>
         <mu2>10000000000000.0</mu2>
         <kp>1000000000.0</kp>
@@ -26,9 +26,9 @@
         <minDepth>0.001</minDepth>
         <maxVel>0.1</maxVel>
-        <fdir1>1 0 0</fdir1>
+        <fdir1>1 0 0</fdir1> -->
     </gazebo>
     <gazebo reference="left_front_wheel_link">
         <material>Gazebo/Grey</material>
-        <mu1>10000000000000.0</mu1>
+        <!-- <mu1>10000000000000.0</mu1>
         <mu2>10000000000000.0</mu2>
         <kp>1000000000.0</kp>
@@ -36,9 +36,9 @@
         <minDepth>0.001</minDepth>
         <maxVel>0.1</maxVel>
-        <fdir1>1 0 0</fdir1>
+        <fdir1>1 0 0</fdir1> -->
     </gazebo>
     <gazebo reference="left_back_wheel_link">
         <material>Gazebo/Grey</material>
-        <mu1>10000000000000.0</mu1>
+        <!-- <mu1>10000000000000.0</mu1>
         <mu2>10000000000000.0</mu2>
         <kp>1000000000.0</kp>
@@ -46,41 +46,55 @@
         <minDepth>0.001</minDepth>
         <maxVel>0.1</maxVel>
-        <fdir1>1 0 0</fdir1>
+        <fdir1>1 0 0</fdir1> -->
     </gazebo>
+<!-- ROS 2 Control -->
     <gazebo>
+    <!-- ROS 2 Humble -->
+        <xacro:if value="$(arg is_ignition)">
         <plugin filename="ign_ros2_control-system" name="ign_ros2_control::IgnitionROS2ControlPlugin">
-            <robot_param>robot_description</robot_param>
-            <robot_param_node>robot_state_publisher</robot_param_node>
             <parameters>$(find my_robot_controller)/config/my_robot_controllers.yaml</parameters>
-            <controller_manager_name>controller_manager</controller_manager_name>
         </plugin>
+        </xacro:if>
+        <!-- ROS 2 Iron or above -->
+        <xacro:unless value="$(arg is_ignition)">
+        <plugin filename="gz_ros2_control-system" name="gz_ros2_control::GazeboSimROS2ControlPlugin">
+            <parameters>$(find my_robot_controller)/config/my_robot_controllers.yaml</parameters>
+        </plugin>
+        </xacro:unless>
     </gazebo>
-    <gazebo reference="lidar_link">
-        <material>Gazebo/Red</material>
-        <sensor name="laser" type="ray">
-            <pose> 0 0 0 0 0 0 </pose>
-            <visualize>true</visualize>
+    <!-- <gazebo reference="lidar_link">
+        <sensor name='gpu_lidar' type='gpu_lidar'>"
+            <topic>scan</topic>
             <update_rate>10</update_rate>
+            <ignition_frame_id>lidar</ignition_frame_id>
             <ray>
                 <scan>
                     <horizontal>
-                        <samples>360</samples>
-                        <min_angle>-3.14</min_angle>
-                        <max_angle>3.14</max_angle>
+                        <samples>3000</samples>
+                        <resolution>0.9</resolution>
+                        <min_angle>-3.1415</min_angle>
+                        <max_angle>3.1415</max_angle>
                     </horizontal>
+                    <vertical>
+                        <samples>1</samples>
+                        <resolution>0.01</resolution>
+                        <min_angle>0</min_angle>
+                        <max_angle>0</max_angle>
+                    </vertical>
                 </scan>
                 <range>
-                    <min>0.3</min>
-                    <max>12</max>
+                    <min>0.15</min>
+                    <max>8.0</max>
+                    <resolution>0.5</resolution>
                 </range>
             </ray>
-            <plugin name="gazebo_ros_head_hokuyo_controller" filename="libgazebo_ros_laser.so">
-                <ros>
-                    <argument>~/out:=scan</argument>
-                </ros>
-                <output_type>sensor_msgs/LaserScan</output_type>
-                <frame_name>laser_frame</frame_name>
-            </plugin>
+            <always_on>1</always_on>
+            <visualize>true</visualize>
         </sensor>
-    </gazebo>
+        <plugin
+            filename="libignition-gazebo-sensors-system.so"
+            name="ignition::gazebo::systems::Sensors">
+            <render_engine>ogre2</render_engine>
+        </plugin>
+    </gazebo> -->
 </robot>

File: my_robot_description/urdf/my_robot_ros2_control.xacro (robot description, xacro)
@@ -2,7 +2,17 @@
 <robot xmlns:xacro="http://www.ros.org/wiki/xacro">
     <ros2_control name="RobotSystem" type="system">
-        <hardware>
-            <plugin>ign_ros2_control/IgnitionSystem</plugin>
-        </hardware>
+        <!-- ros2_control Gazebo -->
+        <!-- ROS 2 Humble -->
+        <xacro:if value="$(arg is_ignition)">
+            <hardware>
+                <plugin>ign_ros2_control/IgnitionSystem</plugin>
+            </hardware>
+        </xacro:if>
+        <!-- ROS 2 Iron or above -->
+        <xacro:unless value="$(arg is_ignition)">
+            <hardware>
+                <plugin>gz_ros2_control/GazeboSimSystem</plugin>
+            </hardware>
+        </xacro:unless>
         <joint name="base_right_front_wheel_joint">
             <command_interface name="velocity">
