Commit message: added IMU (needs testing)

File: my_robot_description/urdf/mobile_base.xacro (robot description, xacro)
@@ -1,11 +1,18 @@
 <?xml version="1.0"?>
 <robot xmlns:xacro="http://www.ros.org/wiki/xacro">
+    <!-- Base -->
     <xacro:property name="base_length" value="0.2" />
     <xacro:property name="base_width" value="0.125" />
     <xacro:property name="base_height" value="0.04" />
+    <!-- Wheels -->
     <xacro:property name="wheel_radius" value="0.034" />
     <xacro:property name="wheel_length" value="0.025" />
+    <!-- Lidar -->
     <xacro:property name="lidar_radius" value="0.036" />
     <xacro:property name="lidar_length" value="0.035" />
+    <!-- IMU -->
+    <xacro:property name="imu_length" value="0.025" />
+    <xacro:property name="imu_width" value="0.025" />
+    <xacro:property name="imu_height" value="0.0025" />
     <link name="base_footprint" />
     <link name="base_link">
@@ -24,5 +31,22 @@
         </collision>
         <xacro:box_inertia m="5.0" l="${2*base_length}" w="${2*base_width}" h="${2*base_height}"
-                           xyz="0 0 ${base_height / 2.0}" rpy="0 0 0" />
+        xyz="0 0 ${base_height / 2.0}" rpy="0 0 0" />
+    </link>
+    <link name="imu_link">
+        <visual>
+            <geometry>
+                <box size="${imu_length} ${imu_width} ${imu_height}" />
+            </geometry>
+            <origin xyz="0 0 ${imu_height / 2.0}" rpy="0 0 0" />
+            <material name="orange" />
+        </visual>
+        <collision>
+            <geometry>
+                <box size="${imu_length} ${imu_width} ${imu_height}" />
+            </geometry>
+            <origin xyz="0 0 ${imu_height / 2.0}" rpy="0 0 0" />
+        </collision>
+        <xacro:box_inertia m="5.0" l="${2*imu_length}" w="${2*imu_width}" h="${2*imu_height}"
+            xyz="0 0 ${imu_height / 2.0}" rpy="0 0 0" />
     </link>
     <link name="lidar_link">
@@ -100,3 +124,9 @@
         <axis xyz="0 1 0" />
     </joint>
+    <joint name="base_imu_joint" type="fixed">
+        <parent link="base_link" />
+        <child link="imu_link" />
+        <origin xyz="${base_length / 2.0 - imu_length} ${base_width / 2.0 - imu_width / 2.0} ${base_height}" rpy="0 0 0" />
+        <axis xyz="0 0 0" />
+    </joint>
 </robot>

File: my_robot_description/urdf/mobile_base_gazebo.xacro (robot description, xacro)
@@ -7,52 +7,29 @@
         <material>Gazebo/Black</material>
     </gazebo>
+    <gazebo reference="imu_link">
+        <material>Gazebo/Orange</material>
+    </gazebo>
     <gazebo reference="right_front_wheel_link">
-        <!-- Buraya bir sey ekledim -->
         <material>Gazebo/Grey</material>
-        <!-- <mu1>10000000000000.0</mu1>
-        <mu2>10000000000000.0</mu2>
-        <kp>1000000000.0</kp>
-        <kd>10.0</kd>
-        <minDepth>0.001</minDepth>
-        <maxVel>0.1</maxVel>
-        <fdir1>1 0 0</fdir1> -->
     </gazebo>
     <gazebo reference="right_back_wheel_link">
         <material>Gazebo/Grey</material>
-        <!-- <mu1>10000000000000.0</mu1>
-        <mu2>10000000000000.0</mu2>
-        <kp>1000000000.0</kp>
-        <kd>10.0</kd>
-        <minDepth>0.001</minDepth>
-        <maxVel>0.1</maxVel>
-        <fdir1>1 0 0</fdir1> -->
     </gazebo>
     <gazebo reference="left_front_wheel_link">
         <material>Gazebo/Grey</material>
-        <!-- <mu1>10000000000000.0</mu1>
-        <mu2>10000000000000.0</mu2>
-        <kp>1000000000.0</kp>
-        <kd>10.0</kd>
-        <minDepth>0.001</minDepth>
-        <maxVel>0.1</maxVel>
-        <fdir1>1 0 0</fdir1> -->
     </gazebo>
     <gazebo reference="left_back_wheel_link">
         <material>Gazebo/Grey</material>
-        <!-- <mu1>10000000000000.0</mu1>
-        <mu2>10000000000000.0</mu2>
-        <kp>1000000000.0</kp>
-        <kd>10.0</kd>
-        <minDepth>0.001</minDepth>
-        <maxVel>0.1</maxVel>
-        <fdir1>1 0 0</fdir1> -->
     </gazebo>
-<!-- ROS 2 Control -->
+    <!-- ROS 2 Control -->
     <gazebo>
     <!-- ROS 2 Humble -->
         <xacro:if value="$(arg is_ignition)">
-        <plugin filename="ign_ros2_control-system" name="ign_ros2_control::IgnitionROS2ControlPlugin">
-            <parameters>$(find my_robot_controller)/config/my_robot_controllers.yaml</parameters>
-        </plugin>
+            <plugin filename="ign_ros2_control-system" name="ign_ros2_control::IgnitionROS2ControlPlugin">
+                <parameters>$(find my_robot_controller)/config/my_robot_controllers.yaml</parameters>
+            </plugin>
+            <plugin filename="ignition-gazebo-sensors-system" name="ignition::gazebo::systems::Sensors">
+                <render_engine>ogre2</render_engine>
+            </plugin>
         </xacro:if>
         <!-- ROS 2 Iron or above -->
@@ -63,38 +40,83 @@
         </xacro:unless>
     </gazebo>
-    <!-- <gazebo reference="lidar_link">
-        <sensor name='gpu_lidar' type='gpu_lidar'>"
+    <gazebo reference="imu_link">
+        <sensor name="imu" type="imu">
+            <always_on>true</always_on>
+            <update_rate>100</update_rate>
+            <gz_frame_id>imu_link</gz_frame_id>
+            <topic>imu</topic>
+            <imu>
+              <angular_velocity>
+                <x>
+                  <noise type="gaussian">
+                    <mean>0.0</mean>
+                    <stddev>2e-4</stddev>
+                  </noise>
+                </x>
+                <y>
+                  <noise type="gaussian">
+                    <mean>0.0</mean>
+                    <stddev>2e-4</stddev>
+                  </noise>
+                </y>
+                <z>
+                  <noise type="gaussian">
+                    <mean>0.0</mean>
+                    <stddev>2e-4</stddev>
+                  </noise>
+                </z>
+              </angular_velocity>
+              <linear_acceleration>
+                <x>
+                  <noise type="gaussian">
+                    <mean>0.0</mean>
+                    <stddev>1.7e-2</stddev>
+                  </noise>
+                </x>
+                <y>
+                  <noise type="gaussian">
+                    <mean>0.0</mean>
+                    <stddev>1.7e-2</stddev>
+                  </noise>
+                </y>
+                <z>
+                  <noise type="gaussian">
+                    <mean>0.0</mean>
+                    <stddev>1.7e-2</stddev>
+                  </noise>
+                </z>
+              </linear_acceleration>
+            </imu>
+        </sensor>
+      </gazebo>
+      <!-- 2D Laser Sensor -->
+    <gazebo reference="lidar_link">
+        <sensor name="lidar" type="gpu_lidar">
+            <always_on>true</always_on>
+            <visualize>true</visualize>
             <topic>scan</topic>
-            <update_rate>10</update_rate>
-            <ignition_frame_id>lidar</ignition_frame_id>
-            <ray>
+            <update_rate>5</update_rate>
+            <gz_frame_id>lidar_link</gz_frame_id>
+            <lidar>
                 <scan>
-                    <horizontal>
-                        <samples>3000</samples>
-                        <resolution>0.9</resolution>
-                        <min_angle>-3.1415</min_angle>
-                        <max_angle>3.1415</max_angle>
-                    </horizontal>
-                    <vertical>
-                        <samples>1</samples>
-                        <resolution>0.01</resolution>
-                        <min_angle>0</min_angle>
-                        <max_angle>0</max_angle>
-                    </vertical>
+                <horizontal>
+                    <samples>360</samples>
+                    <resolution>1.00000</resolution>
+                    <min_angle>0.000000</min_angle>
+                    <max_angle>6.280000</max_angle>
+                </horizontal>
                 </scan>
                 <range>
-                    <min>0.15</min>
-                    <max>8.0</max>
-                    <resolution>0.5</resolution>
+                <min>0.15000</min>
+                <max>8.0</max>
+                <resolution>0.5</resolution>
                 </range>
-            </ray>
-            <always_on>1</always_on>
-            <visualize>true</visualize>
+                <noise>
+                    <type>gaussian</type>
+                    <mean>0.0</mean>
+                    <stddev>0.01</stddev>
+                </noise>
+            </lidar>
         </sensor>
-        <plugin
-            filename="libignition-gazebo-sensors-system.so"
-            name="ignition::gazebo::systems::Sensors">
-            <render_engine>ogre2</render_engine>
-        </plugin>
-    </gazebo> -->
+    </gazebo>
 </robot>

Commit message: ekf added, ekf should be configured (lidar odometry problems)

File: my_robot_description/urdf/mobile_base.xacro (robot description, xacro)
@@ -127,5 +127,5 @@
         <parent link="base_link" />
         <child link="imu_link" />
-        <origin xyz="${base_length / 2.0 - imu_length} ${base_width / 2.0 - imu_width / 2.0} ${base_height}" rpy="0 0 0" />
+        <origin xyz="${base_length / 2.0 - imu_length} ${base_width / 2.0 - imu_width / 2.0} ${base_height}" rpy="3.1415 0 0" />
         <axis xyz="0 0 0" />
     </joint>

File: my_robot_description/urdf/mobile_base_gazebo.xacro (robot description, xacro)
@@ -32,4 +32,5 @@
                 <render_engine>ogre2</render_engine>
             </plugin>
+            <plugin filename="ignition-gazebo-imu-system" name="ignition::gazebo::systems::Imu"></plugin>
         </xacro:if>
         <!-- ROS 2 Iron or above -->

Commit message: ekf options changed, still eneds configuration for IMU

File: my_robot_description/urdf/mobile_base.xacro (robot description, xacro)
@@ -38,5 +38,5 @@
                 <box size="${imu_length} ${imu_width} ${imu_height}" />
             </geometry>
-            <origin xyz="0 0 ${imu_height / 2.0}" rpy="0 0 0" />
+            <origin xyz="0 0 0" rpy="0 0 0" />
             <material name="orange" />
         </visual>
@@ -45,5 +45,5 @@
                 <box size="${imu_length} ${imu_width} ${imu_height}" />
             </geometry>
-            <origin xyz="0 0 ${imu_height / 2.0}" rpy="0 0 0" />
+            <origin xyz="0 0 0" rpy="0 0 0" />
         </collision>
         <xacro:box_inertia m="5.0" l="${2*imu_length}" w="${2*imu_width}" h="${2*imu_height}"
@@ -55,5 +55,5 @@
                   <cylinder radius="${lidar_radius}" length = "${lidar_length}"/>
               </geometry>
-              <origin xyz="0 0 ${lidar_length}" rpy="0 0 0"/>
+              <origin xyz="0 0 0" rpy="0 0 0"/>
               <material name="black"/>
           </visual>
@@ -62,5 +62,5 @@
                 <cylinder radius="${lidar_radius}" length = "${lidar_length}"/>
             </geometry>
-            <origin xyz="0 0 ${lidar_length}" rpy="0 0 0"/>
+            <origin xyz="0 0 0" rpy="0 0 0"/>
           </collision>
     </link>
@@ -121,11 +121,11 @@
         <parent link="base_link" />
         <child link="lidar_link" />
-        <origin xyz="0 0 ${base_height / 2.0}" rpy="0 0 0" />
-        <axis xyz="0 1 0" />
+        <origin xyz="0 0 ${base_height + lidar_length / 2.0}" rpy="0 0 0" />
+        <axis xyz="0 0 0" />
     </joint>
     <joint name="base_imu_joint" type="fixed">
         <parent link="base_link" />
         <child link="imu_link" />
-        <origin xyz="${base_length / 2.0 - imu_length} ${base_width / 2.0 - imu_width / 2.0} ${base_height}" rpy="3.1415 0 0" />
+        <origin xyz="${base_length / 2.0 - imu_length} ${base_width / 2.0 - imu_width / 2.0} ${base_height + imu_height / 2.0}" rpy="0 0 0" />
         <axis xyz="0 0 0" />
     </joint>

File: my_robot_description/urdf/my_robot_ros2_control.xacro (robot description, xacro)
@@ -1,5 +1,5 @@
 <?xml version="1.0"?>
 <robot xmlns:xacro="http://www.ros.org/wiki/xacro">
-    <ros2_control name="RobotSystem" type="system">
+    <ros2_control name="RobotSystem" type="actuator">
         <!-- ros2_control Gazebo -->
         <!-- ROS 2 Humble -->
@@ -20,6 +20,5 @@
                 <param name="max">1</param>
             </command_interface>
-            <state_interface name="position"/>
-            <state_interface name="velocity"/>
+            <state_interface name="position">0</state_interface>
         </joint>
         <joint name="base_right_back_wheel_joint">
@@ -29,6 +28,5 @@
                 <param name="max">1</param>
             </command_interface>
-            <state_interface name="position"/>
-            <state_interface name="velocity"/>
+            <state_interface name="position">0</state_interface>
         </joint>
         <joint name="base_left_front_wheel_joint">
@@ -37,6 +35,5 @@
                 <param name="max">1</param>
             </command_interface>
-            <state_interface name="position"/>
-            <state_interface name="velocity"/>
+            <state_interface name="position">0</state_interface>
         </joint>
         <joint name="base_left_back_wheel_joint">
@@ -45,6 +42,5 @@
                 <param name="max">1</param>
             </command_interface>
-            <state_interface name="position"/>
-            <state_interface name="velocity"/>
+            <state_interface name="position">0</state_interface>
         </joint>
     </ros2_control>

Commit message: worked on hardware interface

File: my_robot_description/urdf/mobile_base.xacro (robot description, xacro)
@@ -122,5 +122,5 @@
         <child link="lidar_link" />
         <origin xyz="0 0 ${base_height + lidar_length / 2.0}" rpy="0 0 0" />
-        <axis xyz="0 0 0" />
+        <axis xyz="0 0 {3.1415/2.0}" />
     </joint>
     <joint name="base_imu_joint" type="fixed">

File: my_robot_description/urdf/mobile_base_gazebo.xacro (robot description, xacro)
@@ -97,5 +97,5 @@
             <visualize>true</visualize>
             <topic>scan</topic>
-            <update_rate>5</update_rate>
+            <update_rate>20</update_rate>
             <gz_frame_id>lidar_link</gz_frame_id>
             <lidar>

File: my_robot_description/urdf/my_robot.urdf.xacro (robot description, xacro)
@@ -1,4 +1,5 @@
 <?xml version="1.0"?>
 <robot name="my_robot" xmlns:xacro="http://www.ros.org/wiki/xacro">
+    <xacro:arg name="is_sim" default="false"/>
     <!-- Properties -->
     <xacro:include filename="common_properties.xacro" />

File: my_robot_description/urdf/my_robot_ros2_control.xacro (robot description, xacro)
@@ -3,16 +3,24 @@
     <ros2_control name="RobotSystem" type="actuator">
         <!-- ros2_control Gazebo -->
-        <!-- ROS 2 Humble -->
-        <xacro:if value="$(arg is_ignition)">
+        <xacro:if value="$(arg is_sim)">
+            <!-- <xacro:if value="$(arg is_ignition)">
+                <hardware>
+                    <plugin>ign_ros2_control/IgnitionSystem</plugin>
+                </hardware>
+            </xacro:if>
+            <xacro:unless value="$(arg is_ignition)">
+                <hardware>
+                    <plugin>gz_ros2_control/GazeboSimSystem</plugin>
+                </hardware>
+            </xacro:unless> -->
+        </xacro:if>
+        <xacro:unless value="$(arg is_sim)">
             <hardware>
-                <plugin>ign_ros2_control/IgnitionSystem</plugin>
-            </hardware>
-        </xacro:if>
-        <!-- ROS 2 Iron or above -->
-        <xacro:unless value="$(arg is_ignition)">
-            <hardware>
-                <plugin>gz_ros2_control/GazeboSimSystem</plugin>
+                <plugin>ros2_control_hardware/DCMotorHardwareInterface</plugin>
+                <param name="wheel_separation">0.15</param>
+                <param name="wheel_radius">0.034</param>
             </hardware>
         </xacro:unless>
+        <!-- ROS 2 Humble -->
         <joint name="base_right_front_wheel_joint">
             <command_interface name="velocity">
@@ -22,12 +30,11 @@
             <state_interface name="position">0</state_interface>
         </joint>
-        <joint name="base_right_back_wheel_joint">
+        <!-- <joint name="base_right_back_wheel_joint">
             <command_interface name="velocity">
-                <!-- I Changed this file -->
                 <param name="min">-1</param>
                 <param name="max">1</param>
             </command_interface>
             <state_interface name="position">0</state_interface>
-        </joint>
+        </joint> -->
         <joint name="base_left_front_wheel_joint">
             <command_interface name="velocity">
@@ -37,5 +44,5 @@
             <state_interface name="position">0</state_interface>
         </joint>
-        <joint name="base_left_back_wheel_joint">
+        <!-- <joint name="base_left_back_wheel_joint">
             <command_interface name="velocity">
                 <param name="min">-1</param>
@@ -43,5 +50,5 @@
             </command_interface>
             <state_interface name="position">0</state_interface>
-        </joint>
+        </joint> -->
     </ros2_control>
 </robot>
